Commit message: Added lidar and cam, but cam processing pending

File: description/robot.urdf.xacro (robot description, xacro)
@@ -2,3 +2,6 @@
 <robot xmlns:xacro="http://www.ros.org/wiki/xacro"  name="robot">
    <xacro:include filename="robot_core.xacro" />
+   <xacro:include filename="gazebo_control.xacro" />
+   <xacro:include filename="lidar.xacro" />
+   <xacro:include filename="camera.xacro" />
 </robot>

File: description/robot_core.xacro (robot description, xacro)
@@ -1,111 +1,128 @@
 <?xml version="1.0"?>
-<robot xmlns:xacro="http://www.ros.org/wiki/xacro" >
-    <xacro:include filename="inertial_macros.xacro" />
-    <material name="white">
-        <color rgba="1 1 1 1"/>
-    </material>
-    <material name="orange">
-        <color rgba="1 0.3 0.1 1"/>
-    </material>
-    <material name="blue">
-        <color rgba="0.2 0.2 1 1"/>
-    </material>
-    <material name="black">
-        <color rgba="0 0 0 1"/>
-    </material>
-    <!-- BASE LINK -->
-    <link name="base_link">
-    </link>
-    <!-- CHASSIS LINK -->
-    <joint name="chassis_joint" type="fixed">
-        <parent link="base_link"/>
-        <child link="chassis"/>
-        <origin xyz="-0.1 0 0"/>
-    </joint>
-    <link name="chassis">
-         <visual>
-               <origin xyz="0.15 0 0.075"/>
-              <geometry>
-                 <box size="0.3 0.3 0.15"/>
-              </geometry>
-              <material name="white"/>
-         </visual>
-         <collision>
-               <origin xyz="0.15 0 0.075"/>
-              <geometry>
-                 <box size="0.3 0.3 0.15"/>
-              </geometry>
-         </collision>
-         <xacro:inertial_box mass="0.5" x="0.3" y="0.3" z="0.15">
-            <origin xyz="0.15 0 0.02" rpy="0 0 0"/><!--z=0.075-->
-         </xacro:inertial_box>
-    </link>
-      <!-- LEFT WHEEL LINK-->
-      <joint name="left_wheel_joint" type="continuous">
-        <parent link="base_link"/>
-        <child link="left_wheel"/>
-        <origin xyz="0 0.175 0" rpy="-${pi/2} 0 0"/>
-        <axis xyz="0 0 1"/>
-    </joint>
-    <link name="left_wheel">
-        <visual>
-            <geometry>
-                <cylinder radius="0.05" length="0.04"/>
-            </geometry>
-            <material name="blue"/>
-        </visual>
-        <collision>
-            <geometry>
-                <cylinder radius="0.05" length="0.04"/>
-            </geometry>
-        </collision>
-        <xacro:inertial_cylinder mass="0.1" length="0.04" radius="0.05">
-           <origin xyz="0 0 0" rpy="0 0 0"/>
-        </xacro:inertial_cylinder>
-    </link>
-    <!-- RIGHT WHEEL LINK-->
-    <joint name="right_wheel_joint" type="continuous">
-        <parent link="base_link"/>
-        <child link="right_wheel"/>
-        <origin xyz="0 -0.175 0" rpy="${pi/2} 0 0"/>
-        <axis xyz="0 0 -1"/>
-    </joint>
-    <link name="right_wheel">
-        <visual>
-            <geometry>
-                <cylinder radius="0.05" length="0.04"/>
-            </geometry>
-            <material name="blue"/>
-        </visual>
-        <collision>
-            <geometry>
-                <cylinder radius="0.05" length="0.04"/>
-            </geometry>
-        </collision>
-        <xacro:inertial_cylinder mass="0.1" length="0.04" radius="0.05">
-           <origin xyz="0 0 0" rpy="0 0 0"/>
-        </xacro:inertial_cylinder>
-    </link>
-    <!-- CASTER WHEEL LINK -->
-    <joint name="caster_wheel_link" type="fixed">
-        <parent link="chassis"/>
-        <child link="caster_wheel"/>
-        <origin xyz="0.24 0 0"/>
-    </joint>
-    <link name="caster_wheel">
-        <visual>
-            <geometry>
-                <sphere radius="0.05"/>
-            </geometry>
-            <material name="black"/>
-        </visual>
-        <collision>
-            <geometry>
-                <sphere radius="0.05"/>
-            </geometry>
-        </collision>
-        <xacro:inertial_sphere mass="0.1" radius="0.05">
-           <origin xyz="0 0 0" rpy="0 0 0"/>
-        </xacro:inertial_sphere>
-    </link>
+<robot xmlns:xacro="http://www.ros.org/wiki/xacro"  >
+<xacro:include filename="inertial_macros.xacro"/>
+<material name="white">
+    <color rgba="1 1 1 1" />
+</material>
+<material name="orange">
+    <color rgba="1 0.3 0.1 1" />
+</material>
+<material name="blue">
+    <color rgba="0.2 0.2 1 1" />
+</material>
+<material name="black">
+    <color rgba="0 0 0 1" />
+</material>
+<material name="red">
+    <color rgba="1 0 0 1" />
+</material>
+<!--base link-->
+<link name="base_link">
+</link>
+ <!--chassis link-->
+<joint name="chassis_joint" type="fixed">
+    <parent link="base_link"/>
+    <child link="chassis"/>
+    <origin xyz="-0.1 0 0"/>
+</joint>
+<link name="chassis">
+     <visual>
+           <origin xyz="0.15 0 0.075"/>
+          <geometry>
+             <box size="0.3 0.3 0.15"/>
+          </geometry>
+          <material name="white"/>
+     </visual>
+     <collision>
+           <origin xyz="0.15 0 0.075"/>
+          <geometry>
+             <box size="0.3 0.3 0.15"/>
+          </geometry>
+     </collision>
+     <xacro:inertial_box mass="0.5" x="0.3" y="0.3" z="0.15">
+        <origin xyz="0.15 0 0.02" rpy="0 0 0"/><!--z=0.075-->
+     </xacro:inertial_box>
+</link>
+<gazebo reference="chassis">
+       <material>Gazebo/White</material>
+</gazebo>
+<!--left wheel link-->
+<joint name="left_wheel_joint" type="continuous">
+          <parent link="base_link"/>
+          <child link="left_wheel"/>
+          <origin xyz="0 0.175 0" rpy="-${pi/2} 0 0"/>
+          <axis xyz="0 0 1"/>
+</joint>
+<link name="left_wheel">
+     <visual>
+       <geometry>
+         <cylinder radius="0.05" length="0.04"/>
+       </geometry>
+       <material name="blue"/>
+    </visual>
+    <collision>
+       <geometry>
+         <cylinder radius="0.05" length="0.04"/>
+       </geometry>
+    </collision>
+    <xacro:inertial_cylinder mass="0.1" length="0.04" radius="0.05">
+       <origin xyz="0 0 0" rpy="0 0 0"/>
+    </xacro:inertial_cylinder>
+</link>
+<gazebo reference="left_wheel">
+       <material>Gazebo/Blue</material>
+</gazebo>
+<!--right wheel link-->
+<joint name="right_wheel_joint" type="continuous">
+          <parent link="base_link"/>
+          <child link="right_wheel"/>
+          <origin xyz="0 -0.175 0" rpy="${pi/2} 0 0"/>
+          <axis xyz="0 0 -1"/>
+</joint>
+<link name="right_wheel">
+     <visual>
+       <geometry>
+         <cylinder radius="0.05" length="0.04"/>
+       </geometry>
+       <material name="blue"/>
+    </visual>
+    <collision>
+       <geometry>
+         <cylinder radius="0.05" length="0.04"/>
+       </geometry>
+    </collision>
+    <xacro:inertial_cylinder mass="0.1" length="0.04" radius="0.05">
+       <origin xyz="0 0 0" rpy="0 0 0"/>
+    </xacro:inertial_cylinder>
+</link>
+<gazebo reference="right_wheel">
+       <material>Gazebo/Blue</material>
+   </gazebo>
+<!--caster wheel link-->
+<joint name="caster_wheel_joint" type="fixed">
+    <parent link="chassis"/>
+    <child link="caster_wheel"/>
+    <origin xyz="0.24 0 0"/>
+</joint>
+<link name="caster_wheel">
+   <visual>
+        <geometry>
+          <sphere radius="0.05"/>
+        </geometry>
+        <material name="black"/>
+   </visual>
+   <collision>
+        <geometry>
+          <sphere radius="0.05"/>
+        </geometry>
+   </collision>
+   <xacro:inertial_sphere mass="0.1" radius="0.05">
+       <origin xyz="0 0 0" rpy="0 0 0"/>
+    </xacro:inertial_sphere>
+</link>
+<gazebo reference="caster_wheel">
+       <material>Gazebo/Black</material>
+       <mu1 value="0.001"/>
+       <mu2 value="0.001"/>
+   </gazebo>
 </robot>
